File: hardware/Wearloc interface/Interface.sch (EAGLE design)
At the start: 44 parts, among them SW1 SSK-1202, U1 PCA9306DCT, U2 LTC2804-1GN, U3 TXB0104D, U4 MCP1826ADJ

Commit message: First routing attempt.
Parts:
- removed PH1_LRP: S3B-XH-A90°, wearloc:S3B-XH-A90°
- removed PH2_LRP, PH_IMU: S4B-XH-A90°, wearloc:S4B-XH-A90°
- removed PH_LH: S6B-XH-A90°, wearloc:S6B-XH-A90°
- removed USB1: MOLEX-47346-0001, wearloc:MOLEX-47346-0001
- added C14: 220µF, rcl:CPOL-EUE3.5-8
- added J1: S7B-XH-A90°, wearloc:S7B-XH-A90°
- added J2: S4B-XH-A90°, wearloc:S4B-XH-A90°
- added J3: S6B-XH-A90°, wearloc:S6B-XH-A90°
- added J4: S2B-XH-A90°, wearloc:S2B-XH-A90°
- C1, C3: value 1µF -> 220nF
- C11: value 100pF -> 4.7µF
- C4, C5: value 220nF -> 1µF
- C9: value 4.7µF -> 100pF
- R10: value 20k 1% -> 1k5
- R11, R7: value 10k -> 1k
- R12, R2: value 1k -> 10k
- R13: device rcl:R-EU_M0805 -> rcl:R-EU_R0805
- R14: value 200 -> 180k 1%
- R15: value 10k -> 20k 1%
- R3: value 1k -> 200
- R4, R5: value 1k5 -> 10k
- R6: value 348k -> 1k
- R8: value 10k -> 348k
- R9: value 180k 1% -> 1k5
- U1: value PCA9306DCT -> LTC2804-1GN; device wearloc:PCA9306DCT -> wearloc:LTC2804-1GN
- U2: value LTC2804-1GN -> PCA9306DCT; device wearloc:LTC2804-1GN -> wearloc:PCA9306DCT
Connections:
- net +1V8: now also C1.2, C6.2, R3.2, R6.1, R7.1, U1.VL, U2.VREF1; no longer C11.2, C4.2, R14.2, R2.1, R3.1, U1.VREF1, U2.VL
- net +4.1V: now also C11.2, R14.2; no longer C10.2, R9.2
- net +5V: now also C10.1, C14.+, C2.2, J1.1, J1.4, J2.3, J3.6, J4.1, R10.2, R11.1, R12.2, R9.2, U1.VCC; no longer C3.2, C9.1, PH1_LRP.1, PH2_LRP.1, PH_IMU.3, PH_LH.6, R12.1, R4.2, R5.2, R6.2, U2.VCC, USB1.1
- net GND: now also C1.1, C10.2, C14.-, C2.1, C4.2, C5.2, C6.1, J1.3, J1.7, J2.4, J3.2, J3.5, J4.2, R15.2, R2.1, R4.1, R5.1; no longer C1.2, C10.1, C2.2, C3.1, C4.1, C6.2, PH1_LRP.3, PH2_LRP.4, PH_IMU.4, PH_LH.2, PH_LH.5, R10.2, R11.1, R15.1, R7.1, USB1.5, USB1.SHIELD
- net I2C_SCL_ED: now also R7.2, U2.SCL1; no longer R2.2, U1.SCL1
- net I2C_SCL_IMU: now also J2.1, R9.1, U2.SCL2; no longer PH_IMU.1, R4.1, U1.SCL2
- net I2C_SDA_ED: now also R6.2, U2.SDA1; no longer R3.2, U1.SDA1
- net I2C_SDA_IMU: now also J2.2, R10.1, U2.SDA2; no longer PH_IMU.2, R5.1, U1.SDA2
- net LH_OUT: now also J3.1, R11.2; no longer PH_LH.1, R12.2
- net MOTOCTL: now also J1.2, U3.B1; no longer PH1_LRP.2, U3.B3
- net N$10: now also R5.2, U1.R2IN; no longer R7.2, U2.R2IN
- net N$11: now also TP2.TP, U1.T2OUT; no longer TP1.TP, U2.T2OUT
- net N$12: now also TP1.TP, U1.R2OUT; no longer TP2.TP, U2.R2OUT
- net N$2: now also R12.1; no longer R8.1
- net N$3: now also R3.1; no longer R14.1
- net N$4: now also R14.1, R15.1; no longer R10.1, R9.1
- net N$5: now also C3.1, U1.SW; no longer C5.1, U2.SW
- net N$6: now also C9.1, R8.1, U2.ENABLE, U2.VREF2; no longer C6.1, R6.1, U1.ENABLE, U1.VREF2
- net N$7: now also C3.2, U1.CAP; no longer C5.2, U2.CAP
- net N$8: now also U1.T2IN; no longer U2.T2IN
- net ON/OFF_RS232: now also R2.2, U1.ON/!OFF; no longer R11.2, U2.ON/!OFF
- net ON/OFF_UART: now also R4.2; no longer R15.2
- net PWM_MOTOCTL_ED: now also U3.A1; no longer U3.A3
- net RS232_RX_LH: now also J3.3, U1.T1OUT; no longer PH_LH.3, U2.T1OUT
- net RS232_TX_LH: now also J3.4, U1.R1IN; no longer PH_LH.4, U2.R1IN
- net UART_RX_ED: now also U1.R1OUT; no longer U2.R1OUT
- net UART_RX_LRP: now also J1.6, U3.B3; no longer PH2_LRP.3, U3.B1
- net UART_TX_ED: now also U1.T1IN, U3.A3; no longer U2.T1IN, U3.A1
- net UART_TX_LRP: now also J1.5; no longer PH2_LRP.2
- net VDD: now also C4.1, U1.VDD; no longer C1.1, U2.VDD
- net VEE: now also C5.1, U1.VEE; no longer C2.1, U2.VEE
Other:
- moved on the sheet: BAT1, C1, C10, C12, C13, C2, C3, C4, C5, C6, D1, R11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

Commit message: almost finished schematic
Parts:
- added R16, R17, R18: 0R, rcl:R-EU_R1206
- R10, R6, R7, R9: device rcl:R-EU_R0805 -> rcl:R-EU_R1206
Connections:
- new net N$13: JP1J18.7, R17.1
- new net N$14: R17.2, R18.1
- new net UART_RX_ED1: R16.2, U3.A2
- net PWM_MOTOCTL_ED: now also R18.2; no longer JP1J18.7
- net UART_RX_ED: now also R16.1; no longer U3.A2
Changed lines of the file:
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@@
 <grid distance="0.1" unitdist="inch" unit="inch" style="lines" multiple="1" display="no" altdistance="0.01" altunitdist="inch" altunit="inch"/>
 <layers>
-<layer number="1" name="Top" color="4" fill="1" visible="no" active="no"/>
-<layer number="16" name="Bottom" color="1" fill="1" visible="no" active="no"/>
-<layer number="17" name="Pads" color="2" fill="1" visible="no" active="no"/>
-<layer number="18" name="Vias" color="2" fill="1" visible="no" active="no"/>
-<layer number="19" name="Unrouted" color="6" fill="1" visible="no" active="no"/>
-<layer number="20" name="Dimension" color="15" fill="1" visible="no" active="no"/>
-<layer number="21" name="tPlace" color="7" fill="1" visible="no" active="no"/>
-<layer number="22" name="bPlace" color="7" fill="1" visible="no" active="no"/>
-<layer number="23" name="tOrigins" color="15" fill="1" visible="no" active="no"/>
-<layer number="24" name="bOrigins" color="15" fill="1" visible="no" active="no"/>
-<layer number="25" name="tNames" color="7" fill="1" visible="no" active="no"/>
-<layer number="26" name="bNames" color="7" fill="1" visible="no" active="no"/>
-<layer number="27" name="tValues" color="7" fill="1" visible="no" active="no"/>
-<layer number="28" name="bValues" color="7" fill="1" visible="no" active="no"/>
+<layer number="1" name="Top" color="4" fill="1" visible="yes" active="no"/>
+<layer number="16" name="Bottom" color="1" fill="1" visible="yes" active="no"/>
+<layer number="17" name="Pads" color="2" fill="1" visible="yes" active="no"/>
+<layer number="18" name="Vias" color="2" fill="1" visible="yes" active="no"/>
+<layer number="19" name="Unrouted" color="6" fill="1" visible="yes" active="no"/>
+<layer number="20" name="Dimension" color="15" fill="1" visible="yes" active="no"/>
+<layer number="21" name="tPlace" color="7" fill="1" visible="yes" active="no"/>
+<layer number="22" name="bPlace" color="7" fill="1" visible="yes" active="no"/>
+<layer number="23" name="tOrigins" color="15" fill="1" visible="yes" active="no"/>
+<layer number="24" name="bOrigins" color="15" fill="1" visible="yes" active="no"/>
+<layer number="25" name="tNames" color="7" fill="1" visible="yes" active="no"/>
+<layer number="26" name="bNames" color="7" fill="1" visible="yes" active="no"/>
+<layer number="27" name="tValues" color="7" fill="1" visible="yes" active="no"/>
+<layer number="28" name="bValues" color="7" fill="1" visible="yes" active="no"/>
 <layer number="29" name="tStop" color="7" fill="3" visible="no" active="no"/>
 <layer number="30" name="bStop" color="7" fill="6" visible="no" active="no"/>
@@
 <layer number="35" name="tGlue" color="7" fill="4" visible="no" active="no"/>
 <layer number="36" name="bGlue" color="7" fill="5" visible="no" active="no"/>
-<layer number="37" name="tTest" color="7" fill="1" visible="no" active="no"/>
-<layer number="38" name="bTest" color="7" fill="1" visible="no" active="no"/>
+<layer number="37" name="tTest" color="7" fill="1" visible="yes" active="no"/>
+<layer number="38" name="bTest" color="7" fill="1" visible="yes" active="no"/>
 <layer number="39" name="tKeepout" color="4" fill="11" visible="no" active="no"/>
 <layer number="40" name="bKeepout" color="1" fill="11" visible="no" active="no"/>
@@
 <layer number="44" name="Drills" color="7" fill="1" visible="no" active="no"/>
 <layer number="45" name="Holes" color="7" fill="1" visible="no" active="no"/>
-<layer number="46" name="Milling" color="3" fill="1" visible="no" active="no"/>
-<layer number="47" name="Measures" color="7" fill="1" visible="no" active="no"/>
-<layer number="48" name="Document" color="7" fill="1" visible="no" active="no"/>
-<layer number="49" name="Reference" color="7" fill="1" visible="no" active="no"/>
-<layer number="50" name="dxf" color="7" fill="1" visible="no" active="no"/>
-<layer number="51" name="tDocu" color="7" fill="1" visible="no" active="no"/>
-<layer number="52" name="bDocu" color="7" fill="1" visible="no" active="no"/>
-<layer number="53" name="tGND_GNDA" color="7" fill="9" visible="no" active="no"/>
-<layer number="54" name="bGND_GNDA" color="1" fill="9" visible="no" active="no"/>
-<layer number="56" name="wert" color="7" fill="1" visible="no" active="no"/>
-<layer number="57" name="tCAD" color="7" fill="1" visible="no" active="no"/>
+<layer number="46" name="Milling" color="3" fill="1" visible="yes" active="no"/>
+<layer number="47" name="Measures" color="7" fill="1" visible="yes" active="no"/>
+<layer number="48" name="Document" color="7" fill="1" visible="yes" active="no"/>
+<layer number="49" name="Reference" color="7" fill="1" visible="yes" active="no"/>
+<layer number="50" name="dxf" color="7" fill="1" visible="yes" active="no"/>
+<layer number="51" name="tDocu" color="7" fill="1" visible="yes" active="no"/>
+<layer number="52" name="bDocu" color="7" fill="1" visible="yes" active="no"/>
+<layer number="53" name="tGND_GNDA" color="7" fill="9" visible="yes" active="no"/>
+<layer number="54" name="bGND_GNDA" color="1" fill="9" visible="yes" active="no"/>
+<layer number="56" name="wert" color="7" fill="1" visible="yes" active="no"/>
+<layer number="57" name="tCAD" color="7" fill="1" visible="yes" active="no"/>
 <layer number="90" name="Modules" color="5" fill="1" visible="yes" active="yes"/>
 <layer number="91" name="Nets" color="2" fill="1" visible="yes" active="yes"/>
@@
 <part name="C7" library="rcl" deviceset="C-EU" device="C0805K" value="100nF"/>
 <part name="C8" library="rcl" deviceset="C-EU" device="C0805K" value="100nF"/>
-<part name="R7" library="rcl" deviceset="R-EU_" device="R0805" value="1k"/>
-<part name="R6" library="rcl" deviceset="R-EU_" device="R0805" value="1k"/>
-<part name="R9" library="rcl" deviceset="R-EU_" device="R0805" value="1k5"/>
-<part name="R10" library="rcl" deviceset="R-EU_" device="R0805" value="1k5"/>
+<part name="R7" library="rcl" deviceset="R-EU_" device="R1206" value="1k"/>
+<part name="R6" library="rcl" deviceset="R-EU_" device="R1206" value="1k"/>
+<part name="R9" library="rcl" deviceset="R-EU_" device="R1206" value="1k5"/>
+<part name="R10" library="rcl" deviceset="R-EU_" device="R1206" value="1k5"/>
 <part name="R8" library="rcl" deviceset="R-EU_" device="R0805" value="348k"/>
 <part name="FRAME1" library="frames" deviceset="A4L-LOC" device="" value="Logic converters"/>
@@
 <part name="C14" library="rcl" deviceset="CPOL-EU" device="E3.5-8" value="220µF"/>
 <part name="P+10" library="supply1" deviceset="+5V" device=""/>
+<part name="R16" library="rcl" deviceset="R-EU_" device="R1206" value="0R"/>
+<part name="R17" library="rcl" deviceset="R-EU_" device="R1206" value="0R"/>
+<part name="R18" library="rcl" deviceset="R-EU_" device="R1206" value="0R"/>
 </parts>
 <sheets>
@@
 <label x="45.72" y="43.18" size="1.27" layer="95" rot="R180" xref="yes"/>
 </segment>
-<segment>
-<pinref part="U3" gate="TXB0104" pin="A2"/>
-<wire x1="162.56" y1="50.8" x2="160.02" y2="50.8" width="0.1524" layer="91"/>
-<label x="160.02" y="50.8" size="1.27" layer="95" rot="R180" xref="yes"/>
-</segment>
 </net>
 <net name="UART_TX_ED" class="0">
@@
 <wire x1="162.56" y1="55.88" x2="160.02" y2="55.88" width="0.1524" layer="91"/>
 <label x="160.02" y="55.88" size="1.27" layer="95" rot="R180" xref="yes"/>
+</segment>
+</net>
+<net name="UART_RX_ED1" class="0">
+<segment>
+<pinref part="U3" gate="TXB0104" pin="A2"/>
+<wire x1="162.56" y1="50.8" x2="160.02" y2="50.8" width="0.1524" layer="91"/>
+<label x="160.02" y="50.8" size="1.27" layer="95" rot="R180" xref="yes"/>
 </segment>
 </net>
@@
 <attribute name="VALUE" x="91.44" y="91.44" size="1.778" layer="96" rot="R180"/>
 </instance>
+<instance part="R16" gate="G$1" x="48.26" y="96.52"/>
+<instance part="R17" gate="G$1" x="66.04" y="111.76"/>
+<instance part="R18" gate="G$1" x="78.74" y="111.76"/>
 </instances>
 <busses>
@@
 </segment>
 </net>
-<net name="UART_RX_ED" class="0">
-<segment>
-<pinref part="JP1" gate="J18" pin="13"/>
-<wire x1="35.56" y1="96.52" x2="43.18" y2="96.52" width="0.1524" layer="91"/>
-<label x="43.18" y="96.52" size="1.27" layer="95" xref="yes"/>
-</segment>
-</net>
 <net name="UART_TX_ED" class="0">
 <segment>
@@
 <net name="PWM_MOTOCTL_ED" class="0">
 <segment>
-<pinref part="JP1" gate="J18" pin="7"/>
-<wire x1="35.56" y1="111.76" x2="43.18" y2="111.76" width="0.1524" layer="91"/>
-<label x="43.18" y="111.76" size="1.27" layer="95" xref="yes"/>
+<label x="86.36" y="111.76" size="1.27" layer="95" xref="yes"/>
+<pinref part="R18" gate="G$1" pin="2"/>
+<wire x1="83.82" y1="111.76" x2="86.36" y2="111.76" width="0.1524" layer="91"/>
 </segment>
 </net>
@@
 </segment>
 </net>
+<net name="UART_RX_ED" class="0">
+<segment>
+<pinref part="JP1" gate="J18" pin="13"/>
+<pinref part="R16" gate="G$1" pin="1"/>
+<wire x1="35.56" y1="96.52" x2="43.18" y2="96.52" width="0.1524" layer="91"/>
+<wire x1="43.18" y1="96.52" x2="43.18" y2="101.6" width="0.1524" layer="91"/>
+<wire x1="43.18" y1="101.6" x2="55.88" y2="101.6" width="0.1524" layer="91"/>
+<label x="55.88" y="101.6" size="1.27" layer="95" xref="yes"/>
+<junction x="43.18" y="96.52"/>
+</segment>
+</net>
+<net name="UART_RX_ED1" class="0">
+<segment>
+<pinref part="R16" gate="G$1" pin="2"/>
+<wire x1="53.34" y1="96.52" x2="55.88" y2="96.52" width="0.1524" layer="91"/>
+<label x="55.88" y="96.52" size="1.27" layer="95" xref="yes"/>
+</segment>
+</net>
+<net name="N$13" class="0">
+<segment>
+<pinref part="R17" gate="G$1" pin="1"/>
+<pinref part="JP1" gate="J18" pin="7"/>
+<wire x1="35.56" y1="111.76" x2="60.96" y2="111.76" width="0.1524" layer="91"/>
+</segment>
+</net>
+<net name="N$14" class="0">
+<segment>
+<pinref part="R17" gate="G$1" pin="2"/>
+<pinref part="R18" gate="G$1" pin="1"/>
+<wire x1="73.66" y1="111.76" x2="71.12" y2="111.76" width="0.1524" layer="91"/>
+</segment>
+</net>
