File: hardware/Wearloc interface/Interface.brd (EAGLE design)
At the start: 100 x 80 mm, 44 parts, among them J1 S7B-XH-A90°, J2 S4B-XH-A90°, J3 S6B-XH-A90°, J4 S2B-XH-A90°, SW1 SSK-1202, U1 LTC2804-1GN, U2 PCA9306DCT, U3 TXB0104D, U4 MCP1826ADJ

Commit message: almost finished schematic
Parts:
- added R16, R17, R18: 0R, rcl:R1206
- R10, R6, R7, R9: device rcl:R0805 -> rcl:R1206
- moved R9 135.6 mm to (55.9, 19.5), flipped to the bottom
- moved R6 132.7 mm to (53.5, 34.3), flipped to the bottom, turned to 90 degrees
- moved C2 128.2 mm to (40.2, 16.7), flipped to the bottom, turned to 180 degrees
- moved R5 122.6 mm to (47.5, 21.4), flipped to the bottom
- moved C9 117.2 mm to (55.6, 25.9), flipped to the bottom, turned to 90 degrees
- moved C6 111.2 mm to (56.7, 31.1), flipped to the bottom, turned to 180 degrees
- moved R1 107.3 mm to (47.5, 25.2), flipped to the bottom, turned to 180 degrees
- moved TP2 107.0 mm to (43.3, 16.8), flipped to the bottom
- moved R10 99.0 mm to (57.3, 16.4), flipped to the bottom
- moved L1 97.0 mm to (40.2, 18.6), flipped to the bottom
- moved TP1 95.7 mm to (44.6, 30.0), flipped to the bottom
- moved C4 90.7 mm to (47.5, 23.3), flipped to the bottom, turned to 180 degrees
- moved R8 90.4 mm to (55.7, 21.9), flipped to the bottom
- moved R4 89.1 mm to (9.05, 16.5), flipped to the bottom
- moved C3 88.0 mm to (38.6, 23.5), flipped to the bottom, turned to 90 degrees
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Connections:
- new net N$13: JP1.J18_7, R17.1
- new net N$14: R17.2, R18.1
- new net UART_RX_ED1: R16.2, U3.3
- net PWM_MOTOCTL_ED: now also R18.2; no longer JP1.J18_7
- net UART_RX_ED: now also R16.1; no longer U3.3
Routing:
- net GND: track 76.7 -> 408.7 mm, vias 0 -> 12
- net +5V: track 22.6 -> 206.2 mm, vias 0 -> 4
- net +1V8: track 0.00 -> 105.0 mm, vias 0 -> 4
- net I2C_SCL_ED: track 0.00 -> 68.5 mm
- net I2C_SDA_ED: track 0.00 -> 68.5 mm
- net UART_TX_ED: track 0.00 -> 57.0 mm
- net N$1: track 0.00 -> 47.2 mm
- net ON/OFF_RS232: track 0.00 -> 44.8 mm
- net UART_RX_ED: track 0.00 -> 40.8 mm
- net LH_OUT_ED: track 0.00 -> 40.2 mm
- net UART_RX_ED1: track 0.00 -> 32.2 mm
- net N$13: track 0.00 -> 29.7 mm
- net ON/OFF_UART: track 0.00 -> 28.8 mm
- net LH_OUT: track 0.00 -> 20.6 mm
- net I2C_SCL_IMU: track 0.00 -> 16.4 mm
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- added copper zone on layer 1, net GND
- added copper zone on layer 16, net GND
- added copper zone on layer 1, net N$15
- added copper zone on layer 1, net N$16
- added copper zone on layer 1, net N$17
Other:
- board size 100 x 80 mm -> 80 x 70 mm

Commit message: small changes in board layout
Routing:
- net GND: vias 12 -> 14
Changed lines of the file:
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@@
 <wire x1="30.48" y1="47.625" x2="27.94" y2="45.085" width="1.016" layer="1"/>
 <wire x1="27.94" y1="45.085" x2="27.94" y2="41.275" width="1.016" layer="1"/>
+<via x="3.81" y="66.675" extent="1-16" drill="1" diameter="1.9304" shape="octagon"/>
+<via x="64.77" y="66.675" extent="1-16" drill="1" diameter="1.9304" shape="octagon"/>
 </signal>
 <signal name="N$6">
